Commit message: added camera and costmap improvement

File: rbcar_common/rbcar_description/robots/rbcar.urdf.xacro (robot description, xacro)
@@ -11,5 +11,5 @@
 	<!-- Import all available sensors -->
 	<xacro:include filename="$(find robotnik_sensors)/urdf/all_sensors.urdf.xacro" />
-        <xacro:include filename="$(find velodyne_description)/urdf/VLP-16.urdf.xacro"/>
+	<xacro:include filename="$(find velodyne_description)/urdf/VLP-16.urdf.xacro"/>
 	<!-- ***************** -->
 	<!-- Global parameters -->
@@ -49,6 +49,6 @@
 		<origin xyz="0.0 0.0 0.170" rpy="0 0 0"/>
 	</xacro:sensor_imu>
-        <xacro:VLP-16 parent="base_link" name="velodyne" topic="/velodyne_points" hz="10" samples="440">
-		<origin xyz="-0.17 0 2.0" rpy="0 0 0"/>
+  <xacro:VLP-16 parent="base_link" name="velodyne" topic="/velodyne_points" hz="10" samples="440">
+		<origin xyz="0.3 0 2.0" rpy="0 0 0"/>
 	</xacro:VLP-16>
 	<!-- xacro:sensor_hokuyo_utm30lx name="hokuyo" parent="base_link">
@@ -71,9 +71,7 @@
 	</xacro:sensor_asus_xtion_pro>
 -->
-<!--
-	<xacro:sensor_kinect name="kinect" parent="base_link">
-		<origin xyz="0.3 0.0 0.16" rpy="0 0 0"/>
+	<xacro:sensor_kinect prefix="kinect" parent="base_link">
+		<origin xyz="0.9 0.0 1.7" rpy="0 0 0"/>
 	</xacro:sensor_kinect>
--->
 <!--
 	<xacro:sensor_fotonic name="fotonic" parent="base_link">
