Commit message: shifted zed camera

File: car_description/urdf/nv11.urdf.xacro (robot description, xacro)
@@ -33,5 +33,5 @@
 	<!-- Put in Sensors -->
 	<!-- <xacro:zed_camera parent="base_link">
-		<origin xyz="-0.788 0 1.176" rpy="0 0 0"/>
+		<origin xyz="0.68778 0 0.380" rpy="0 0 0" />
 	</xacro:zed_camera> -->
 	<!-- <xacro:vlp16 name="vlp16" parent="base_link">
@@ -39,5 +39,5 @@
 	</xacro:vlp16> -->
 	<xacro:ti_radar parent="base_link">
-		<origin xyz=" 0.68778 0 0.380" rpy="0 0 0" />
+		<origin xyz="0.68778 0 0.380" rpy="0 0 0" />
 	</xacro:ti_radar>
 	<!-- simulated sensors -->
@@ -46,5 +46,5 @@
 	</xacro:sensor_imu>
 	<xacro:sensor_kinect prefix="zed" parent="base_link">
-		<origin xyz="-0.788 0 1.176" rpy="0 0 0"/>
+		<origin xyz="0.68778 0 0.380" rpy="0 0 0" />
 	</xacro:sensor_kinect>
 	<xacro:VLP-16 parent="base_link" name="velodyne" topic="/velodyne_points" hz="10" samples="440">-->

Commit message: tuned to smooth motion

File: car_description/urdf/nv11.urdf.xacro (robot description, xacro)
@@ -35,10 +35,10 @@
 		<origin xyz="0.68778 0 0.380" rpy="0 0 0" />
 	</xacro:zed_camera> -->
-	<!-- <xacro:vlp16 name="vlp16" parent="base_link">
-		<origin xyz="0 1.381 1.22877" rpy="0 0 0" />
-	</xacro:vlp16> -->
+	<!--<xacro:vlp16 name="vlp16" parent="base_link">
+		<origin xyz="-1.381 0 1.22877" rpy="0 0 0" />
+	</xacro:vlp16>
 	<xacro:ti_radar parent="base_link">
 		<origin xyz="0.68778 0 0.380" rpy="0 0 0" />
-	</xacro:ti_radar>
+	</xacro:ti_radar>-->
 	<!-- simulated sensors -->
 	<xacro:sensor_imu prefix="imu" parent="base_link">
@@ -49,5 +49,5 @@
 	</xacro:sensor_kinect>
 	<xacro:VLP-16 parent="base_link" name="velodyne" topic="/velodyne_points" hz="10" samples="440">-->
-		<origin xyz="0 0 1.22877" rpy="0 0 0" />
+		<origin xyz="-1.381 0 1.22877" rpy="0 0 0" />
 	</xacro:VLP-16>
 </robot>

File: car_description/urdf/wheels/car_wheels.urdf.xacro (robot description, xacro)
@@ -10,5 +10,5 @@
   <xacro:property name="tire_width" value="0.095"/>
   <xacro:property name="hex_hub_depth" value="0.05223"/> <!-- or +0.072 -->
-  <xacro:property name="wheel_mass" value="8.0"/>   <!-- check -->
+  <xacro:property name="wheel_mass" value="3.3"/>   <!-- check -->
   <!-- hex_hub_dist is the distance between left and right hex hubs when
        the shock absorbers are fully extended. axle_length is the distance
@@ -45,5 +45,5 @@
        measured in rad/s. -->
   <xacro:property name="servo_stall_torque" value="50"/>  <!-- check -->
-  <xacro:property name="servo_no_load_speed" value="25"/> <!-- check -->
+  <xacro:property name="servo_no_load_speed" value="50"/> <!-- check -->
   <!-- Inertia of a thick-walled cylindrical tube with open ends. Height is
        measured along the z axis, which is the tube's axis. inner_rad and
