Commit message: modified model

File: car_description/urdf/wheels/car_wheels.urdf.xacro (robot description, xacro)
@@ -17,8 +17,9 @@
   <xacro:property name="wheelbase" value="2.07"/>
   <xacro:property name="hex_hub_dist" value="1.06296"/>  <!-- 1.127 0.742 0.900 check -->
-  <xacro:property name="axle_length" value="0"/>
+  <xacro:property name="axle_length" value="0.12"/>
   <xacro:property name="wheel_travel" value="0"/>
   <xacro:property name="shock_z_offset" value="0.00"/>
   <!-- Degree-to-radian conversions -->
+  <xacro:property name="degrees_30" value="0.523599" />
   <xacro:property name="degrees_45" value="0.785398163"/>
   <xacro:property name="degrees_90" value="1.57079633"/>
@@ -170,5 +171,5 @@
       <child link="${lr_prefix}_${fr_prefix}_axle_carrier"/>
       <axis xyz="0 0 1"/>
-      <limit lower="${-degrees_45}" upper="${degrees_45}"
+      <limit lower="${-degrees_30}" upper="${degrees_30}"
              effort="${servo_stall_torque}" velocity="${servo_no_load_speed}"/>
     </joint>

Commit message: updated steering limits

File: car_description/urdf/wheels/car_wheels.urdf.xacro (robot description, xacro)
@@ -21,4 +21,5 @@
   <xacro:property name="shock_z_offset" value="0.00"/>
   <!-- Degree-to-radian conversions -->
+  <xacro:property name="degrees_20" value="0.349066" />
   <xacro:property name="degrees_30" value="0.523599" />
   <xacro:property name="degrees_45" value="0.785398163"/>
@@ -171,5 +172,5 @@
       <child link="${lr_prefix}_${fr_prefix}_axle_carrier"/>
       <axis xyz="0 0 1"/>
-      <limit lower="${-degrees_30}" upper="${degrees_30}"
+      <limit lower="${-degrees_20}" upper="${degrees_20}"
              effort="${servo_stall_torque}" velocity="${servo_no_load_speed}"/>
     </joint>

Commit message: adjusted urdf to stop jerking

File: car_description/urdf/wheels/car_wheels.urdf.xacro (robot description, xacro)
@@ -30,7 +30,7 @@
   <xacro:property name="shock_vel_limit" value="1000"/>
   <xacro:property name="wheel_joint_damping" value="0.2" />
-  <xacro:property name="wheel_joint_friction" value="0.3" />
-  <xacro:property name="suspension_joint_damping" value="0.0" />
-  <xacro:property name="suspension_joint_friction" value="0.0" />
+  <xacro:property name="wheel_joint_friction" value="0.7" />
+  <xacro:property name="suspension_joint_damping" value="0.2" />
+  <xacro:property name="suspension_joint_friction" value="0.7" />
   <!-- axle eff limit = 2 * stall_torque
        as a function of the max gradient (15%) with overall max payload (600Kg) * wheel_radius

Commit message: zach

File: car_description/urdf/wheels/car_wheels.urdf.xacro (robot description, xacro)
@@ -45,5 +45,5 @@
        measured in rad/s. -->
   <xacro:property name="servo_stall_torque" value="50"/>  <!-- check -->
-  <xacro:property name="servo_no_load_speed" value="50"/> <!-- check -->
+  <xacro:property name="servo_no_load_speed" value="25"/> <!-- check -->
   <!-- Inertia of a thick-walled cylindrical tube with open ends. Height is
        measured along the z axis, which is the tube's axis. inner_rad and
