Commit message: Cleaned up files and changed base link weight to be at the center

File: car_description/urdf/bases/car_base.urdf.xacro (robot description, xacro)
@@ -6,5 +6,5 @@
     <xacro:property name="PI" value="3.1415926535897931"/>
     <!-- TODO: CHANGE WHEEL WIDTH -->
-    <xacro:property name="wheel_width" value="0.175" />
+    <xacro:property name="wheel_width" value="0.275" />
     <xacro:property name="clearance" value="0" />
     <!-- BASE FOOTPRINT -->
@@ -19,5 +19,5 @@
         </link>
         <joint name="base_footprint_joint" type="fixed">
-        <origin xyz="0 0 ${clearance}" rpy="0 0 0" />  <!-- height is the clearance -->
+        <origin xyz="0 0 ${clearance}" rpy="0 0 0" />
         <parent link="base_footprint"/>
         <child link="base_link" />
@@ -27,7 +27,7 @@
     <link name="base_link">
         <inertial>
-        <origin xyz="0 0 0" rpy="0 0 0" />
+        <origin xyz="-1.1 0 0" rpy="0 0 0" />
         <mass value="230" />
-        <inertia
+         <inertia
             ixx="0.93313"
             ixy="-0.17064"
@@ -40,5 +40,6 @@
         <origin xyz="0 0 0" rpy="0 0 0" />
         <geometry>
-            <mesh filename="package://car/meshes/base_link.STL" />
+             <mesh filename="package://car/meshes/base_link.STL" />
+	    <box size="0.001 0.001 0.001" />
         </geometry>
         <material name="">
@@ -49,5 +50,5 @@
         <origin xyz="0 0 0" rpy="0 0 0" />
         <geometry>
-            <mesh filename="package://car/meshes/base_link.STL" />
+            <box size="0.001 0.001 0.001" />
         </geometry>
         </collision>

File: car_description/urdf/nv11.urdf.xacro (robot description, xacro)
@@ -6,5 +6,4 @@
 	<!-- Sensors -->
 	<xacro:include filename="$(find car)/urdf/sensors/zed_camera.urdf.xacro" />
-	<xacro:include filename="$(find car)/urdf/sensors/vlp16.urdf.xacro" />
 	<xacro:include filename="$(find car)/urdf/sensors/ti_radar.urdf.xacro" />
 	<xacro:include filename="$(find velodyne_description)/urdf/VLP-16.urdf.xacro"/>
@@ -49,6 +48,6 @@
 		<origin xyz="-0.788 0 1.176" rpy="0 0 0"/>
 	</xacro:sensor_kinect>
-	<xacro:VLP-16 parent="base_link" name="velodyne" topic="/velodyne_points" hz="10" samples="440">
-		<origin xyz="-1.381 0 1.22877" rpy="0 0 0" />
+	<xacro:VLP-16 parent="base_link" name="velodyne" topic="/velodyne_points" hz="10" samples="440">-->
+		<origin xyz="0 0 1.22877" rpy="0 0 0" />
 	</xacro:VLP-16>
 </robot>

File: car_description/urdf/sensors/ti_radar.urdf.xacro (robot description, xacro)
@@ -9,8 +9,8 @@
     <link name="radar_link">
         <visual>
-            <origin xyz="0 50 50" rpy="0 0 0"/>
-            <geometry>
+            <origin xyz="0 0 1.5" rpy="0 0 0"/>
+            <!--<geometry>
                 <mesh filename="package://car/meshes/lidar.STL" />
-            </geometry>
+            </geometry>-->
             <material name="light_grey">
                 <color rgba="0.8 0.8 0.8 0.8"/>

File: car_description/urdf/wheels/car_wheels.urdf.xacro (robot description, xacro)
@@ -30,7 +30,7 @@
   <xacro:property name="shock_vel_limit" value="1000"/>
   <xacro:property name="wheel_joint_damping" value="0.2" />
-  <xacro:property name="wheel_joint_friction" value="0.7" />
-  <xacro:property name="suspension_joint_damping" value="0" />
-  <xacro:property name="suspension_joint_friction" value="0" />
+  <xacro:property name="wheel_joint_friction" value="0.3" />
+  <xacro:property name="suspension_joint_damping" value="0.0" />
+  <xacro:property name="suspension_joint_friction" value="0.0" />
   <!-- axle eff limit = 2 * stall_torque
        as a function of the max gradient (15%) with overall max payload (600Kg) * wheel_radius

Commit message: changed base link to back

File: car_description/urdf/bases/car_base.urdf.xacro (robot description, xacro)
@@ -12,5 +12,5 @@
         <link name="base_footprint">
         <visual>
-            <origin xyz="0 0 0" rpy="0 0 0" />
+            <origin xyz="-0.01596 0 0" rpy="0 0 0" />
             <geometry>
                 <box size="0.001 0.001 0.001" />
@@ -19,5 +19,5 @@
         </link>
         <joint name="base_footprint_joint" type="fixed">
-        <origin xyz="0 0 ${clearance}" rpy="0 0 0" />
+        <origin xyz="-0.01596 0 ${clearance}" rpy="0 0 0" />
         <parent link="base_footprint"/>
         <child link="base_link" />
@@ -27,16 +27,16 @@
     <link name="base_link">
         <inertial>
-        <origin xyz="-1.1 0 0" rpy="0 0 0" />
-        <mass value="230" />
-         <inertia
-            ixx="0.93313"
-            ixy="-0.17064"
-            ixz="0.0039682"
-            iyy="0.69622"
-            iyz="-0.049966"
-            izz="0.47227" />
+        <origin xyz="0.4 0 0" rpy="0 0 0" />
+        <mass value="192.69" />
+        <inertia
+        ixx="33.169"
+        ixy="-1.105"
+        ixz="-9.0191"
+        iyy="117.15"
+        iyz="1.4735"
+        izz="118.94" />
         </inertial>
         <visual>
-        <origin xyz="0 0 0" rpy="0 0 0" />
+        <origin xyz="2.07 0 0" rpy="0 0 0" />
         <geometry>
              <mesh filename="package://car/meshes/base_link.STL" />
@@ -48,5 +48,4 @@
         </visual>
         <collision>
-        <origin xyz="0 0 0" rpy="0 0 0" />
         <geometry>
             <box size="0.001 0.001 0.001" />

File: car_description/urdf/nv11.urdf.xacro (robot description, xacro)
@@ -24,11 +24,11 @@
 	<!-- Wheels -->
 		<xacro:front_wheel lr_prefix="left" fr_prefix="front"
-						lr_reflect="1" fr_reflect="1" xyz="-0.01596 0.51686 0.24885"/>
+						lr_reflect="1" fr_reflect="1" xyz="2.05404 0.51686 0.24885"/>
 		<xacro:front_wheel lr_prefix="right" fr_prefix="front"
-							lr_reflect="-1" fr_reflect="1" xyz="-0.01596 -0.51686 0.24885"/>
+							lr_reflect="-1" fr_reflect="1" xyz="2.05404 -0.51686 0.24885"/>
 		<xacro:rear_wheel lr_prefix="left" fr_prefix="rear"
-							lr_reflect="1" fr_reflect="-1" xyz="-2.08596 0.51686 0.24885"/>
+							lr_reflect="1" fr_reflect="-1" xyz="-0.01596 0.51686 0.24885"/>
 		<xacro:rear_wheel lr_prefix="right" fr_prefix="rear"
-							lr_reflect="-1" fr_reflect="-1" xyz="-2.08596 -0.51686 0.24885"/>
+							lr_reflect="-1" fr_reflect="-1" xyz="-0.01596 -0.51686 0.24885"/>
 	<!-- Put in Sensors -->
 	<!-- <xacro:zed_camera parent="base_link">
@@ -43,11 +43,11 @@
 	<!-- simulated sensors -->
 	<xacro:sensor_imu prefix="imu" parent="base_link">
-		<origin xyz="0.0 0.0 0.170" rpy="0 0 0"/>
+		<origin xyz="2.07 0.0 0.170" rpy="0 0 0"/>
 	</xacro:sensor_imu>
 	<xacro:sensor_kinect prefix="zed" parent="base_link">
-		<origin xyz="0.68778 0 0.380" rpy="0 0 0" />
+		<origin xyz="2.75778 0 0.380" rpy="0 0 0" />
 	</xacro:sensor_kinect>
 	<xacro:VLP-16 parent="base_link" name="velodyne" topic="/velodyne_points" hz="10" samples="440">-->
-		<origin xyz="-1.381 0 1.22877" rpy="0 0 0" />
+		<origin xyz="0.689 0 1.22877" rpy="0 0 0" />
 	</xacro:VLP-16>
 </robot>

Commit message: fixed recovery drift by correcting wheelbase

File: car_description/urdf/bases/car_base.urdf.xacro (robot description, xacro)
@@ -6,5 +6,5 @@
     <xacro:property name="PI" value="3.1415926535897931"/>
     <!-- TODO: CHANGE WHEEL WIDTH -->
-    <xacro:property name="wheel_width" value="0.275" />
+    <xacro:property name="wheel_width" value="0.095" />
     <xacro:property name="clearance" value="0" />
     <!-- BASE FOOTPRINT -->
@@ -27,6 +27,6 @@
     <link name="base_link">
         <inertial>
-        <origin xyz="0.4 0 0" rpy="0 0 0" />
-        <mass value="192.69" />
+        <origin xyz="0.55 0 0" rpy="0 0 0" />
+        <mass value="1" />
         <inertia
         ixx="33.169"
